Commit message: tests and first refactoring

File: examples/panda.urdf (robot description, URDF)
Before this commit: robot panda, 9 links, 8 joints
Links:
- added link panda_FT, mass 0.0001
- added link world
- link panda_link0: geometry collision cylinder length=0.03 radius=0.06; collision sphere radius=0.06
- link panda_link1: geometry collision cylinder length=0.2830 radius=0.06; collision sphere radius=0.06
- link panda_link2: geometry collision cylinder length=0.12 radius=0.06; collision sphere radius=0.06
- link panda_link3: geometry collision cylinder length=0.15 radius=0.06; collision sphere radius=0.06
- link panda_link4: geometry collision cylinder length=0.12 radius=0.06; collision sphere radius=0.06
- link panda_link5: geometry collision cylinder length=0.1 radius=0.06; collision cylinder length=0.14 radius=0.025
- link panda_link6: geometry collision cylinder length=0.08 radius=0.05; collision sphere radius=0.05
- link panda_link7: geometry collision cylinder length=0.14 radius=0.04; collision sphere radius=0.04
Joints:
- added joint panda_jointFT: type fixed, parent panda_link8, child panda_FT, origin xyz=0 0 0 rpy=0 0 -0.785398163397, axis 0 0 0
- added joint support_to_world: type fixed, parent world, child panda_link0, origin xyz=0.0 0.0 0.0 rpy=0.0 0.0 0.0
