Commit message: FrictionRobotWrapper splitted and few fixes

File: pynocchio/models/urdf/panda.urdf (robot description, URDF)
Before this commit: robot panda, 11 links, 10 joints
Links:
- removed link panda_tool
- added link panda_FT, mass 0.0001
Joints:
- removed joint panda_joint_tool
- added joint panda_jointFT: type fixed, parent panda_link8, child panda_FT, origin xyz=0 0 0 rpy=0 0 -0.785398163397, axis 0 0 0
- joint world_joint: origin xyz=0 -0.6 0 rpy=0 0 0 -> xyz=0 0 0 rpy=0 0 0
